Commit message: change 1400 to 140

File: robot_specific_config/abb_irb1300_7_140_moveit_config/config/abb_irb1300_7_140.ros2_control.xacro (robot description, xacro)
@@ -1,5 +1,5 @@
 <?xml version="1.0"?>
 <robot xmlns:xacro="http://www.ros.org/wiki/xacro">
-    <xacro:macro name="abb_irb1300_7_1400_ros2_control" params="name initial_positions_file">
+    <xacro:macro name="abb_irb1300_7_140_ros2_control" params="name initial_positions_file">
         <xacro:property name="initial_positions" value="${load_yaml(initial_positions_file)['initial_positions']}"/>
         <ros2_control name="${name}" type="system">
